Commit message: sim up

File: simulation/Environment/Weighing/assets/urdf/spoon/spoon.urdf (robot description, URDF)
Before this commit: robot bucket, 5 links, 3 joints
Links:
- link bucket_link: geometry collision mesh filename=Environment/Weighing/assets/urdf/spoon/spoon.stl; visual mesh filename=Environment/Weighing/assets/urdf/spoon/spoon.dae
